File: electroscope_pth.sch (KiCad schematic (older format))
At the start: 19 parts, among them Q1 Q_PNP_BCE, Q2 Q_NPN_BCE, Q3 Q_PNP_BCE, Q4 Q_NPN_BCE, Q5 Q_PNP_BCE, Q6 Q_NPN_BCE, U1 ANT, U2 ANT

Commit message: General placement down
Parts:
- removed D3, D4: LED, ~, symbol LED
- removed Q1, Q3, Q5: Q_PNP_BCE, symbol Q_PNP_BCE
- removed Q2, Q4, Q6: Q_NPN_BCE, symbol Q_NPN_BCE
- added Q1, Q3, Q5: Q_PNP_EBC, symbol Q_PNP_EBC
- added Q2, Q4, Q6: Q_NPN_EBC, symbol Q_NPN_EBC
Connections:
- net GND: now also Q6.1 (E)
- net VCC: now also Q1.1 (E)
- net at R5.1: now also Q5.3 (C)
- net at D2.2 (K): now also Q6.3 (C)
- net at R3.1: now also Q3.3 (C)
- net at R1.1: now also Q1.3 (C)
- net at R2.2: now also Q2.3 (C)
- net at R4.2: now also Q4.3 (C)
- net at U1.1 (IN): now also Q2.2 (B)
- net at U2.1 (IN): now also Q5.2 (B)
- new net: Q2.1 (E), Q4.2 (B)
- new net: Q4.1 (E), Q6.2 (B)
- new net: Q3.2 (B), Q5.1 (E)
- new net: Q1.2 (B), Q3.1 (E)
Changed lines of the file:
@@
 $EndComp
 $Comp
-L GND #PWR4
+L GND #PWR01
 U 1 1 52EEA5AA
 P 4910 5610
-F 0 "#PWR4" H 4910 5610 30  0001 C CNN
+F 0 "#PWR01" H 4910 5610 30  0001 C CNN
 F 1 "GND" H 4910 5540 30  0001 C CNN
 F 2 "" H 4910 5610 60  0000 C CNN
@@
 $EndComp
 $Comp
-L GND #PWR6
+L GND #PWR02
 U 1 1 52EEA5B0
 P 5590 5610
-F 0 "#PWR6" H 5590 5610 30  0001 C CNN
+F 0 "#PWR02" H 5590 5610 30  0001 C CNN
 F 1 "GND" H 5590 5540 30  0001 C CNN
 F 2 "" H 5590 5610 60  0000 C CNN
@@
 $EndComp
 $Comp
-L VCC #PWR1
+L VCC #PWR03
 U 1 1 52EEA725
 P 4270 3180
-F 0 "#PWR1" H 4270 3280 30  0001 C CNN
+F 0 "#PWR03" H 4270 3280 30  0001 C CNN
 F 1 "VCC" H 4270 3280 30  0000 C CNN
 F 2 "" H 4270 3180 60  0000 C CNN
@@
 $EndComp
 $Comp
-L GND #PWR2
+L GND #PWR04
 U 1 1 52EEA74B
 P 4270 3640
-F 0 "#PWR2" H 4270 3640 30  0001 C CNN
+F 0 "#PWR04" H 4270 3640 30  0001 C CNN
 F 1 "GND" H 4270 3570 30  0001 C CNN
 F 2 "" H 4270 3640 60  0000 C CNN
@@
 $EndComp
 $Comp
-L VCC #PWR7
+L VCC #PWR05
 U 1 1 52EEA824
 P 6120 1810
-F 0 "#PWR7" H 6120 1910 30  0001 C CNN
+F 0 "#PWR05" H 6120 1910 30  0001 C CNN
 F 1 "VCC" H 6120 1910 30  0000 C CNN
 F 2 "" H 6120 1810 60  0000 C CNN
@@
 $EndComp
 $Comp
-L VCC #PWR5
+L VCC #PWR06
 U 1 1 52EEA82A
 P 5560 1760
-F 0 "#PWR5" H 5560 1860 30  0001 C CNN
+F 0 "#PWR06" H 5560 1860 30  0001 C CNN
 F 1 "VCC" H 5560 1860 30  0000 C CNN
 F 2 "" H 5560 1760 60  0000 C CNN
@@
 $EndComp
 $Comp
-L VCC #PWR9
+L VCC #PWR07
 U 1 1 52EEA8AC
 P 6720 1840
-F 0 "#PWR9" H 6720 1940 30  0001 C CNN
+F 0 "#PWR07" H 6720 1940 30  0001 C CNN
 F 1 "VCC" H 6720 1940 30  0000 C CNN
 F 2 "" H 6720 1840 60  0000 C CNN
@@
 $EndComp
 $Comp
-L VCC #PWR3
+L VCC #PWR08
 U 1 1 52EEA971
 P 4910 3830
-F 0 "#PWR3" H 4910 3930 30  0001 C CNN
+F 0 "#PWR08" H 4910 3930 30  0001 C CNN
 F 1 "VCC" H 4910 3930 30  0000 C CNN
 F 2 "" H 4910 3830 60  0000 C CNN
@@
 $EndComp
 $Comp
-L GND #PWR8
+L GND #PWR09
 U 1 1 52EEAB28
 P 6330 6220
-F 0 "#PWR8" H 6330 6220 30  0001 C CNN
+F 0 "#PWR09" H 6330 6220 30  0001 C CNN
 F 1 "GND" H 6330 6150 30  0001 C CNN
 F 2 "" H 6330 6220 60  0000 C CNN
@@
 $EndComp
 $Comp
-L GND #PWR10
+L GND #PWR010
 U 1 1 52E1F050
 P 6720 3610
-F 0 "#PWR10" H 6720 3610 30  0001 C CNN
+F 0 "#PWR010" H 6720 3610 30  0001 C CNN
 F 1 "GND" H 6720 3540 30  0001 C CNN
 F 2 "" H 6720 3610 60  0000 C CNN
@@
 	1    0    0    -1
 $EndComp
-$Comp
-L LED D4
-U 1 1 5349D0D7
-P 7050 2750
-F 0 "D4" H 7050 2850 50  0000 C CNN
-F 1 "LED" H 7050 2650 50  0000 C CNN
-F 2 "~" H 7050 2750 60  0000 C CNN
-F 3 "~" H 7050 2750 60  0000 C CNN
-	1    7050 2750
-	0    1    1    0
-$EndComp
-$Comp
-L LED D3
-U 1 1 5349D140
-P 5200 5290
-F 0 "D3" H 5200 5390 50  0000 C CNN
-F 1 "LED" H 5200 5190 50  0000 C CNN
-F 2 "~" H 5200 5290 60  0000 C CNN
-F 3 "~" H 5200 5290 60  0000 C CNN
-	1    5200 5290
-	0    1    1    0
-$EndComp
 Wire Wire Line
 	5560 2900 5560 3000
@@
 	6720 3480 6720 3610
 Wire Wire Line
-	6720 2490 7050 2490
-Wire Wire Line
-	7050 2490 7050 2550
-Connection ~ 6720 2490
-Wire Wire Line
-	6720 3010 7050 3010
-Wire Wire Line
-	7050 3010 7050 2950
-Connection ~ 6720 3010
-Wire Wire Line
-	4910 5040 5200 5040
-Wire Wire Line
-	5200 5040 5200 5090
-Connection ~ 4910 5040
-Wire Wire Line
 	4910 5490 4910 5610
 Wire Wire Line
-	4910 5550 5200 5550
-Wire Wire Line
-	5200 5550 5200 5490
-Connection ~ 4910 5550
-$Comp
-L Q_NPN_BCE Q2
-U 1 1 55EF6D14
-P 5460 2700
-F 0 "Q2" H 5760 2750 50  0000 R CNN
-F 1 "Q_NPN_BCE" H 6060 2650 50  0000 R CNN
-F 2 "" H 5660 2800 29  0000 C CNN
-F 3 "" H 5460 2700 60  0000 C CNN
-	1    5460 2700
-	1    0    0    -1
-$EndComp
-$Comp
-L Q_PNP_BCE Q1
-U 1 1 55EF6E75
-P 5010 4160
-F 0 "Q1" H 5310 4210 50  0000 R CNN
-F 1 "Q_PNP_BCE" H 5610 4110 50  0000 R CNN
-F 2 "" H 5210 4260 29  0000 C CNN
-F 3 "" H 5010 4160 60  0000 C CNN
-	1    5010 4160
-	-1   0    0    1
-$EndComp
-Wire Wire Line
 	4910 4360 4910 4590
 Wire Wire Line
 	4910 4890 4910 5090
-$Comp
-L Q_PNP_BCE Q3
-U 1 1 55EF75E7
-P 5690 4730
-F 0 "Q3" H 5990 4780 50  0000 R CNN
-F 1 "Q_PNP_BCE" H 6290 4680 50  0000 R CNN
-F 2 "" H 5890 4830 29  0000 C CNN
-F 3 "" H 5690 4730 60  0000 C CNN
-	1    5690 4730
-	-1   0    0    1
-$EndComp
 Wire Wire Line
 	5590 4930 5590 5100
@@
 Wire Wire Line
 	6330 5980 6330 6220
-$Comp
-L Q_PNP_BCE Q5
-U 1 1 55EF7C8C
-P 6430 5290
-F 0 "Q5" H 6730 5340 50  0000 R CNN
-F 1 "Q_PNP_BCE" H 7030 5240 50  0000 R CNN
-F 2 "" H 6630 5390 29  0000 C CNN
-F 3 "" H 6430 5290 60  0000 C CNN
-	1    6430 5290
-	-1   0    0    1
-$EndComp
 Wire Wire Line
 	6330 5680 6330 5490
-$Comp
-L Q_NPN_BCE Q4
-U 1 1 55EF8223
-P 6020 3000
-F 0 "Q4" H 6320 3050 50  0000 R CNN
-F 1 "Q_NPN_BCE" H 6620 2950 50  0000 R CNN
-F 2 "" H 6220 3100 29  0000 C CNN
-F 3 "" H 6020 3000 60  0000 C CNN
-	1    6020 3000
-	1    0    0    -1
-$EndComp
-$Comp
-L Q_NPN_BCE Q6
-U 1 1 55EF82C5
-P 6620 3280
-F 0 "Q6" H 6920 3330 50  0000 R CNN
-F 1 "Q_NPN_BCE" H 7220 3230 50  0000 R CNN
-F 2 "" H 6820 3380 29  0000 C CNN
-F 3 "" H 6620 3280 60  0000 C CNN
-	1    6620 3280
-	1    0    0    -1
-$EndComp
 Wire Wire Line
 	6720 2320 6720 2550
@@
 Wire Wire Line
 	5010 2700 5260 2700
+$Comp
+L Q_NPN_EBC Q2
+U 1 1 55F01011
+P 5460 2700
+F 0 "Q2" H 5760 2750 50  0000 R CNN
+F 1 "Q_NPN_EBC" H 6060 2650 50  0000 R CNN
+F 2 "" H 5660 2800 29  0000 C CNN
+F 3 "" H 5460 2700 60  0000 C CNN
+	1    5460 2700
+	1    0    0    -1
+$EndComp
+$Comp
+L Q_NPN_EBC Q4
+U 1 1 55F010A0
+P 6020 3000
+F 0 "Q4" H 6320 3050 50  0000 R CNN
+F 1 "Q_NPN_EBC" H 6620 2950 50  0000 R CNN
+F 2 "" H 6220 3100 29  0000 C CNN
+F 3 "" H 6020 3000 60  0000 C CNN
+	1    6020 3000
+	1    0    0    -1
+$EndComp
+$Comp
+L Q_NPN_EBC Q6
+U 1 1 55F0111A
+P 6620 3280
+F 0 "Q6" H 6920 3330 50  0000 R CNN
+F 1 "Q_NPN_EBC" H 7220 3230 50  0000 R CNN
+F 2 "" H 6820 3380 29  0000 C CNN
+F 3 "" H 6620 3280 60  0000 C CNN
+	1    6620 3280
+	1    0    0    -1
+$EndComp
+$Comp
+L Q_PNP_EBC Q5
+U 1 1 55F011FA
+P 6430 5290
+F 0 "Q5" H 6730 5340 50  0000 R CNN
+F 1 "Q_PNP_EBC" H 7030 5240 50  0000 R CNN
+F 2 "" H 6630 5390 29  0000 C CNN
+F 3 "" H 6430 5290 60  0000 C CNN
+	1    6430 5290
+	-1   0    0    1
+$EndComp
+$Comp
+L Q_PNP_EBC Q3
+U 1 1 55F0123D
+P 5690 4730
+F 0 "Q3" H 5990 4780 50  0000 R CNN
+F 1 "Q_PNP_EBC" H 6290 4680 50  0000 R CNN
+F 2 "" H 5890 4830 29  0000 C CNN
+F 3 "" H 5690 4730 60  0000 C CNN
+	1    5690 4730
+	-1   0    0    1
+$EndComp
+$Comp
+L Q_PNP_EBC Q1
+U 1 1 55F0129D
+P 5010 4160
+F 0 "Q1" H 5310 4210 50  0000 R CNN
+F 1 "Q_PNP_EBC" H 5610 4110 50  0000 R CNN
+F 2 "" H 5210 4260 29  0000 C CNN
+F 3 "" H 5010 4160 60  0000 C CNN
+	1    5010 4160
+	-1   0    0    1
+$EndComp
 $EndSCHEMATC

Commit message: Add updated electroscope schematic
Parts:
- BT1: symbol Battery -> electroscope_pth-rescue:Battery
- D1, D2: symbol LED -> electroscope_pth-rescue:LED
- Q1, Q3, Q5: symbol Q_PNP_EBC -> electroscope_pth-rescue:Q_PNP_EBC
- Q2, Q4, Q6: symbol Q_NPN_EBC -> electroscope_pth-rescue:Q_NPN_EBC
- R1, R2, R3, R4, R5, R6: symbol R -> electroscope_pth-rescue:R
- U1, U2: symbol ANT -> ant:ANT
Changed lines of the file:
@@
-EESchema Schematic File Version 2
-LIBS:power
-LIBS:device
-LIBS:transistors
-LIBS:conn
-LIBS:linear
-LIBS:regul
-LIBS:74xx
-LIBS:cmos4000
-LIBS:adc-dac
-LIBS:memory
-LIBS:xilinx
-LIBS:special
-LIBS:microcontrollers
-LIBS:dsp
-LIBS:microchip
-LIBS:analog_switches
-LIBS:motorola
-LIBS:texas
-LIBS:intel
-LIBS:audio
-LIBS:interface
-LIBS:digital-audio
-LIBS:philips
-LIBS:display
-LIBS:cypress
-LIBS:siliconi
-LIBS:opto
-LIBS:atmel
-LIBS:contrib
-LIBS:valves
-LIBS:ant
+EESchema Schematic File Version 4
 LIBS:electroscope_pth-cache
-EELAYER 25 0
+EELAYER 26 0
 EELAYER END
 $Descr A4 11693 8268
@@
 $EndDescr
 $Comp
-L R R5
+L electroscope_pth-rescue:R R5
 U 1 1 52E1F0B9
 P 6330 5830
@@
 $EndComp
 $Comp
-L LED D2
+L electroscope_pth-rescue:LED D2
 U 1 1 52E1F0CA
 P 6720 2750
@@
 $EndComp
 $Comp
-L R R3
+L electroscope_pth-rescue:R R3
 U 1 1 52E1F193
 P 5590 5250
@@
 $EndComp
 $Comp
-L R R1
+L electroscope_pth-rescue:R R1
 U 1 1 52E1F199
 P 4910 4740
@@
 $EndComp
 $Comp
-L R R2
+L electroscope_pth-rescue:R R2
 U 1 1 52E1F19F
 P 5560 2100
@@
 $EndComp
 $Comp
-L R R4
+L electroscope_pth-rescue:R R4
 U 1 1 52E1F1A5
 P 6120 2130
@@
 $EndComp
 $Comp
-L R R6
+L electroscope_pth-rescue:R R6
 U 1 1 52E1F1AB
 P 6720 2170
@@
 $EndComp
 $Comp
-L LED D1
+L electroscope_pth-rescue:LED D1
 U 1 1 52E1F1B1
 P 4910 5290
@@
 $EndComp
 $Comp
-L GND #PWR01
+L power:GND #PWR01
 U 1 1 52EEA5AA
 P 4910 5610
@@
 $EndComp
 $Comp
-L GND #PWR02
+L power:GND #PWR02
 U 1 1 52EEA5B0
 P 5590 5610
@@
 $EndComp
 $Comp
-L VCC #PWR03
+L power:VCC #PWR03
 U 1 1 52EEA725
 P 4270 3180
@@
 $EndComp
 $Comp
-L GND #PWR04
+L power:GND #PWR04
 U 1 1 52EEA74B
 P 4270 3640
@@
 $EndComp
 $Comp
-L VCC #PWR05
+L power:VCC #PWR05
 U 1 1 52EEA824
 P 6120 1810
@@
 $EndComp
 $Comp
-L VCC #PWR06
+L power:VCC #PWR06
 U 1 1 52EEA82A
 P 5560 1760
@@
 $EndComp
 $Comp
-L VCC #PWR07
+L power:VCC #PWR07
 U 1 1 52EEA8AC
 P 6720 1840
@@
 $EndComp
 $Comp
-L VCC #PWR08
+L power:VCC #PWR08
 U 1 1 52EEA971
 P 4910 3830
@@
 $EndComp
 $Comp
-L GND #PWR09
+L power:GND #PWR09
 U 1 1 52EEAB28
 P 6330 6220
@@
 $EndComp
 $Comp
-L GND #PWR010
+L power:GND #PWR010
 U 1 1 52E1F050
 P 6720 3610
@@
 	6120 2280 6120 2800
 $Comp
-L Battery BT1
+L electroscope_pth-rescue:Battery BT1
 U 1 1 55EF92BC
 P 4270 3420
@@
 	4270 3570 4270 3640
 $Comp
-L ANT U1
+L ant:ANT U1
 U 1 1 55EF983B
 P 5010 1870
@@
 $EndComp
 $Comp
-L ANT U2
+L ant:ANT U2
 U 1 1 55EF9AF0
 P 6970 4400
@@
 	5010 2700 5260 2700
 $Comp
-L Q_NPN_EBC Q2
+L electroscope_pth-rescue:Q_NPN_EBC Q2
 U 1 1 55F01011
 P 5460 2700
@@
 $EndComp
 $Comp
-L Q_NPN_EBC Q4
+L electroscope_pth-rescue:Q_NPN_EBC Q4
 U 1 1 55F010A0
 P 6020 3000
@@
 $EndComp
 $Comp
-L Q_NPN_EBC Q6
+L electroscope_pth-rescue:Q_NPN_EBC Q6
 U 1 1 55F0111A
 P 6620 3280
@@
 $EndComp
 $Comp
-L Q_PNP_EBC Q5
+L electroscope_pth-rescue:Q_PNP_EBC Q5
 U 1 1 55F011FA
 P 6430 5290
@@
 $EndComp
 $Comp
-L Q_PNP_EBC Q3
+L electroscope_pth-rescue:Q_PNP_EBC Q3
 U 1 1 55F0123D
 P 5690 4730
@@
 $EndComp
 $Comp
-L Q_PNP_EBC Q1
+L electroscope_pth-rescue:Q_PNP_EBC Q1
 U 1 1 55F0129D
 P 5010 4160
